File: eagle/v0.2/controller.sch (EAGLE design)
At the start: 7 parts, among them J1 12401832E402A

Commit message: I/O's
Parts:
- added JP4, JP5, JP6, JP7, JP8: (no value), pinhead:PINHD-1X2
- added R1, R2, R3, R4, R5, R6, R7, R8: 10k, rcl:R-EU_R0805
- JP1: device pinhead:PINHD-2X2 -> pinhead:PINHD-1X2
Connections:
- new net A: J1.RX1+, J1.TX1+, JP4.2, R4.1
- new net B: J1.RX1-, J1.TX1-
- new net DOWN: J1.CC2, J1.SBU1
- new net LEFT: J1.RX2-, J1.TX2-
- new net N$1: JP1.2, R1.1
- new net N$11: R1.2, R2.2, R3.2, R4.2, R5.2, R6.2, R7.2, R8.2
- new net N$2: JP2.2, R2.1
- new net N$4: JP3.2, R3.1
- new net N$7: JP8.2, R5.1
- new net N$8: JP7.2, R6.1
- new net N$9: JP6.2, R7.1
- new net RIGHT: J1.RX2+, J1.TX2+
- new net SELECT: J1.D+1, J1.D-2
- new net START: J1.CC1, J1.SBU2
- new net UP: J1.D+2, J1.D-1, JP5.2, R8.1
- net +5V: now also JP1.1, JP2.1, JP3.1, JP4.1, JP5.1, JP6.1, JP7.1, JP8.1
Other:
- moved on the sheet: C1, C9, J1, JP2, JP3, R12
