File: eagle/v0.2/vga.sch (EAGLE design)
At the start: 32 parts, among them J1 12401832E402A, J2 12401832E402A, J3 12401832E402A, J4 12401832E402A, J5 12401832E402A, J7 L77HDE15SD1CH4RHNVGA

Commit message: I/O's
Parts:
- removed C1, C2, C3, C4, C5: 100nF, deto:C1
- removed CPU1, CPU2, GPU1, GPU2: (no value), pinhead:PINHD-1X20
- removed J2, J3, J4, J5: 12401832E402A, Connector_USB:12401832E402A
- removed J6: (no value), SparkFun-Connectors:AUDIO_JACK_2.5MM_2.5MM
- removed J7: L77HDE15SD1CH4RHNVGA, L77HDE15SD1CH4RHNVGA:L77HDE15SD1CH4RHNVGA
- removed R1, R2, R3, R4, R5: Ferrit, deto:R2
- J1: value 12401832E402A -> L77HDE15SD1CH4RHNVGA; device Connector_USB:12401832E402A -> L77HDE15SD1CH4RHNVGA:L77HDE15SD1CH4RHNVGA
Connections:
- removed net +5V: C1.2, C2.2, C3.2, C4.2, C5.2, R1.2, R2.2, R3.2, R4.2, R5.2
- removed net C1_A: J4.RX1+, J4.TX1+
- removed net C1_B: J4.RX1-, J4.TX1-
- removed net C1_DOWN: J4.CC2, J4.SBU1
- removed net C1_LEFT: J4.RX2-, J4.TX2-
- removed net C1_RIGHT: J4.RX2+, J4.TX2+
- removed net C1_SELECT: J4.D+1, J4.D-2
- removed net C1_START: J4.CC1, J4.SBU2
- removed net C1_UP: J4.D+2, J4.D-1
- removed net C2_A: J5.RX1+, J5.TX1+
- removed net C2_B: J5.RX1-, J5.TX1-
- removed net C2_DOWN: J5.CC2, J5.SBU1
- removed net C2_LEFT: J5.RX2-, J5.TX2-
- removed net C2_RIGHT: J5.RX2+, J5.TX2+
- removed net C2_SELECT: J5.D+1, J5.D-2
- removed net C2_START: J5.CC1, J5.SBU2
- removed net C2_UP: J5.D+2, J5.D-1
- removed net C3_A: J2.RX1+, J2.TX1+
- removed net C3_B: J2.RX1-, J2.TX1-
- removed net C3_DOWN: J2.CC2, J2.SBU1
- removed net C3_LEFT: J2.RX2-, J2.TX2-
- removed net C3_RIGHT: J2.RX2+, J2.TX2+
- removed net C3_SELECT: J2.D+1, J2.D-2
- removed net C3_START: J2.CC1, J2.SBU2
- removed net C3_UP: J2.D+2, J2.D-1
- removed net C4_A: J3.RX1+, J3.TX1+
- removed net C4_B: J3.RX1-, J3.TX1-
- removed net C4_DOWN: J3.CC2, J3.SBU1
- removed net C4_LEFT: J3.RX2-, J3.TX2-
- removed net C4_RIGHT: J3.RX2+, J3.TX2+
- removed net C4_SELECT: J3.D+1, J3.D-2
- removed net C4_START: J3.CC1, J3.SBU2
- removed net C4_UP: J3.D+2, J3.D-1
- removed net N$2: J3.VBUS1, J3.VBUS2, J3.VBUS3, J3.VBUS4, R2.1
- removed net N$4: J4.VBUS1, J4.VBUS2, J4.VBUS3, J4.VBUS4, R3.1
- removed net N$6: J7.3, R_BLUE1.2, R_BLUE2.2, R_BLUE3.2
- removed net N$7: J7.1, R_RED1.2, R_RED2.2, R_RED3.2, R_RED4.2
- removed net N$8: J7.2, R_GREEN1.2, R_GREEN2.2, R_GREEN3.2, R_GREEN4.2
- removed net SHIELD4: J1.SHIELD1, J1.SHIELD2, J1.SHIELD3, J1.SHIELD4, J2.SHIELD1, J2.SHIELD2, J2.SHIELD3, J2.SHIELD4, J3.SHIELD1, J3.SHIELD2, J3.SHIELD3, J3.SHIELD4, J4.SHIELD1, J4.SHIELD2, J4.SHIELD3, J4.SHIELD4, J5.SHIELD1, J5.SHIELD2, J5.SHIELD3, J5.SHIELD4
- net GND: now also J1.10, J1.5, J1.6, J1.7, J1.8; no longer C1.1, C2.1, C3.1, C4.1, C5.1, J1.GND1, J1.GND2, J1.GND3, J1.GND4, J2.GND1, J2.GND2, J2.GND3, J2.GND4, J3.GND1, J3.GND2, J3.GND3, J3.GND4, J4.GND1, J4.GND2, J4.GND3, J4.GND4, J5.GND1, J5.GND2, J5.GND3, J5.GND4, J7.10, J7.5, J7.6, J7.7, J7.8
- net HSYNC: now also J1.13; no longer J7.13
- net N$1: now also J1.2, R_GREEN1.2, R_GREEN2.2, R_GREEN3.2, R_GREEN4.2; no longer J2.VBUS1, J2.VBUS2, J2.VBUS3, J2.VBUS4, R1.1
- net N$3: now also J1.3, R_BLUE1.2, R_BLUE2.2, R_BLUE3.2; no longer J1.VBUS1, J1.VBUS2, J1.VBUS3, J1.VBUS4, R5.1
- net N$5: now also J1.1, R_RED1.2, R_RED2.2, R_RED3.2, R_RED4.2; no longer J5.VBUS1, J5.VBUS2, J5.VBUS3, J5.VBUS4, R4.1
- net VSYNC: now also J1.14; no longer J7.14
