File: eagle/mainboard.brd (EAGLE design)
At the start: 100 x 100 mm, 92 parts, among them IC1 74HC02D, IC2 74HC151D, IC3 74HC151D, IC4 74HC590D

Commit message: Work in progress board rework
Parts:
- removed C12, C13, C14, C15, C16, C17, C18, C19, C20, C21, C22, C23: 100nF, rcl:C0805
- removed C_DATA_1, C_DATA_2, C_DATA_3, C_DATA_4: (no value), pinhead:1X03
- added CLOCK1: (no value), pinhead:1X01
- moved R23 39.8 mm to (17.2, 36.7)
- moved C6 16.5 mm to (30.6, 57.5)
- moved R56 16.1 mm to (22.4, 55.3), flipped to the top, turned to 0 degrees
- moved R54 14.4 mm to (28.7, 54.4), turned to 90 degrees
- moved R20 14.3 mm to (70.3, 53.9), flipped to the bottom, turned to 0 degrees
- moved 3V3 14.3 mm to (81.1, 49.2)
- moved SD-CARD 13.5 mm to (25.0, 54.6), flipped to the top, turned to 180 degrees
- moved R16 9.42 mm to (64.3, 50.6), flipped to the bottom, turned to 90 degrees
- moved R19 9.40 mm to (69.2, 50.6), flipped to the bottom, turned to 90 degrees
- moved R18 9.40 mm to (66.7, 50.6), flipped to the bottom, turned to 90 degrees
- moved R13 9.16 mm to (36.2, 50.9), flipped to the bottom, turned to 90 degrees
- moved R14 9.16 mm to (33.6, 50.9), flipped to the bottom, turned to 90 degrees
- moved R11 9.16 mm to (38.7, 50.9), flipped to the bottom, turned to 90 degrees
- moved R9 7.74 mm to (49.0, 58.7), flipped to the bottom, turned to 270 degrees
- moved R8 7.73 mm to (46.4, 58.7), flipped to the bottom, turned to 270 degrees
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Connections:
- net C1: no longer C_DATA_1.2
- net C1_DATA: no longer C_DATA_1.1
- net C2: no longer C_DATA_2.2
- net C2_DATA: no longer C_DATA_2.1
- net C3: no longer C_DATA_3.2
- net C3_DATA: no longer C_DATA_3.1
- net C4: no longer C_DATA_4.2
- net C4_DATA: no longer C_DATA_4.1
- net CONTROLLER_OUT: now also CLOCK1.1
- net DOUBLE1: no longer C21.1
- net DOUBLE2: no longer C23.1
- net GND: no longer C12.2, C13.2, C14.2, C15.2, C16.2, C17.2, C18.2, C19.2, C20.2, C21.2, C22.2, C23.2
- net HOT_PLUG1: no longer C20.1
- net HOT_PLUG2: no longer C22.1
- net ID0_1: no longer C15.1
- net ID0_2: no longer C19.1
- net ID1_1: no longer C14.1
- net ID1_2: no longer C18.1
- net ID2_1: no longer C13.1
- net ID2_2: no longer C17.1
- net ID3_1: no longer C12.1
- net ID3_2: no longer C16.1
Routing:
- net ID3_2: track 116.5 -> 42.3 mm
- net VGA_GREEN: track 81.9 -> 10.8 mm, vias 2 -> 0
- net ID2_2: track 113.5 -> 43.2 mm
- net VGA_RED: track 72.9 -> 3.32 mm
- net HOT_PLUG1: track 115.5 -> 48.0 mm, vias 2 -> 1
- net ID1_2: track 110.5 -> 44.2 mm
- net ID0_2: track 107.5 -> 45.2 mm
- net DOUBLE1: track 100.7 -> 40.4 mm, vias 2 -> 1
- net GPU_MOSI: track 19.8 -> 65.5 mm
- net VGA_BLUE: track 50.5 -> 9.52 mm, vias 2 -> 0
- net C_CLOCK: track 78.8 -> 38.3 mm
- net PA8_CPU: track 3.50 -> 41.4 mm, vias 0 -> 1
- net HOT_PLUG2: track 89.9 -> 59.4 mm
- net DOUBLE2: track 79.9 -> 49.7 mm
- net HSYNC: track 86.3 -> 61.0 mm
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Other:
- outline, holes or cut-outs redrawn
