File: eagle/mainboard.sch (EAGLE design)
At the start: 122 parts, among them IC1 74HCT151D, IC2 74HC04D, IC4 74HCT151D, IC7 74HC590D

Commit message: Schematic complete
Parts:
- removed CPU2, GPU1: (no value), pinhead:PINHD-1X20
- removed IC7: 74HC590D, 74xx-eu:74HC590D
- added C10, C11, C8, C9: 100nF, rcl:C-EUC0805
- added IC3: 74HC151D, 74xx-eu:74HC151D
- CPU, GPU: device pinhead:PINHD-1X20 -> BluePill:BLUE_PILLADVANCED
- IC1: value 74HCT151D -> 74HC02D; device 74xx-eu:74HCT151D -> 74xx-eu:74HC02D
- IC2: value 74HC04D -> 74HC151D; device 74xx-eu:74HC04D -> 74xx-eu:74HC151D
- IC4: value 74HCT151D -> 74HC590D; device 74xx-eu:74HCT151D -> 74xx-eu:74HC590D
Connections:
- removed net CLOCK: CONTROLLER-IN.DN1, IC7A.CLK, IC7A.RCK, JP14.1
- removed net N$19: JP3.2, R63.1
- removed net N$20: JP13.2, R65.1
- removed net N$22: JP12.2, R66.1
- removed net N$23: JP11.2, R67.1
- removed net N$28: IC1A.W
- removed net PB12_CPU: CPU.1, SD-CARD.CD/DAT3
- removed net PB13_CPU: CPU.2, SD-CARD.CLK
- removed net PB14_CPU: CPU.3, R56.1, SD-CARD.DAT0
- removed net PB15_CPU: CPU.4, SD-CARD.CMD
- removed net PC14_CPU: CPU2.3, R54.1, SD-CARD.CD
- new net CONTROLLER_CLOCK: CONTROLLER-IN.DN1, IC4A.CLK, IC4A.RCK, JP14.1
- new net GNDA: C10.2, C11.2, C8.2, C9.2, IC1D.I0, IC1D.I1, IC1P.GND, IC2A.D0, IC2A.D1, IC2A.D2, IC2A.D3, IC2A.D4, IC2A.D5, IC2A.D6, IC2P.GND, IC3P.GND, IC4A.CCKEN, IC4A.G, IC4P.GND, R61.2, R62.2, R63.2, R64.2, R65.2, R66.2, R67.2, R68.2
- new net SDCARDCLK: CPU.PB13, SD-CARD.CLK
- new net SDCARDCMD: CPU.PB15, SD-CARD.CMD
- new net SDCARDHOTPLUG: CPU.PC14, R54.1, SD-CARD.CD
- new net SDCARDIN: CPU.PB12, SD-CARD.CD/DAT3
- new net SDCARDOUT: CPU.PB14, R56.1, SD-CARD.DAT0
- new net VCC: C10.1, C11.1, C7.2, C8.1, C9.1, IC1P.VCC, IC2A.D7, IC2P.VCC, IC3P.VCC, IC4A.CCLR, IC4P.VCC, JP1.1, JP10.1, JP11.1, JP12.1, JP13.1, JP2.1, JP3.1, JP9.1, R71.2
- net +3V3: now also CPU.3.3V, CPU.3.3V1, GPU.3.3V, GPU.3.3V1; no longer CPU.20, CPU2.18, GPU.18, GPU1.20, IC1A.D7
- net +5V: now also CPU.5V, GPU.5V; no longer C7.2, CPU.18, GPU1.18, IC7A.CCLR, JP1.1, JP10.1, JP11.1, JP12.1, JP13.1, JP2.1, JP3.1, JP9.1, R71.2
- net A: now also IC3A.D7; no longer IC4A.D7
- net B: now also IC3A.D6, JP3.2, R63.1; no longer IC4A.D6
- net BLUE_LSP: now also GPU.PB5; no longer GPU1.13
- net BLUE_MMSP: now also GPU.PB6; no longer GPU1.14
- net BLUE_MSP: now also GPU.PB7; no longer GPU1.15
- net CONTROLLER_OUT: now also IC1C.O; no longer IC1A.Y, IC4A.Y
- net DOWN: now also IC3A.D2, JP11.2, R67.1; no longer IC4A.D2
- net GND: now also CPU.GND, CPU.GND1, CPU.GND2, GPU.GND, GPU.GND1, GPU.GND2; no longer CPU.19, CPU2.19, CPU2.20, GPU.19, GPU.20, GPU1.19, IC1A.D0, IC1A.D1, IC1A.D2, IC1A.D3, IC1A.D4, IC1A.D5, IC1A.D6, IC2B.I, IC2C.I, IC2D.I, IC2E.I, IC2F.I, IC7A.CCKEN, IC7A.G
- net GPU_MISO: now also CPU.PB4, GPU.PA6; no longer CPU.12, GPU.11
- net GPU_MOSI: now also CPU.PB5, GPU.PA7; no longer CPU.13, GPU.12
- net GPU_READY: now also CPU.PC15, GPU.PC15; no longer CPU2.4, GPU.4
- net GPU_SCK: now also CPU.PB3, GPU.PA5; no longer CPU.11, GPU.10
- net GPU_SS: now also CPU.PA15, GPU.PA4; no longer CPU.10, GPU.9
- net GREEN_LSP: now also GPU.PB14; no longer GPU1.3
- net GREEN_MMSP: now also GPU.PB13; no longer GPU1.2
- net GREEN_MSP: now also GPU.PB12; no longer GPU1.1
- net HSYNC: now also GPU.PA8; no longer GPU1.5
- net LEFT: now also IC3A.D1, JP12.2, R66.1; no longer IC4A.D1
- net N$11: now also IC1B.I0, IC2A.Y; no longer R61.2, R62.2, R63.2, R64.2, R65.2, R66.2, R67.2, R68.2
- net N$15: now also IC1B.I1, IC3A.Y; no longer JP1.2, R61.1
- net N$17: now also IC1B.O, IC1C.I0, IC1C.I1; no longer JP2.2, R62.1
- net N$24: now also IC2A.C, IC3A.A, IC4A.QA; no longer IC1A.C, IC4A.A, IC7A.QA
- net N$25: now also IC2A.B, IC3A.B, IC4A.QB; no longer IC1A.B, IC4A.B, IC7A.QB
- net N$26: now also IC2A.A, IC3A.C, IC4A.QC; no longer IC1A.A, IC4A.C, IC7A.QC
- net N$27: now also IC1A.I0, IC1A.I1, IC2A.G, IC4A.QD; no longer IC1A.G, IC2A.I, IC7A.QD
- net N$29: now also IC1A.O, IC3A.G; no longer IC2A.O, IC4A.G
- net PA0_GPU: now also GPU.PA0; no longer GPU.5
- net PA10_CPU: now also CPU.PA10; no longer CPU.7
- net PA10_CPU1: now also CPU.PA12; no longer CPU.9
- net PA10_CPU2: now also CPU.PA2; no longer CPU2.7
- net PA10_CPU3: now also CPU.PA0; no longer CPU2.5
- net PA10_CPU4: now also CPU.PA6; no longer CPU2.11
- net PA10_CPU5: now also CPU.PA4; no longer CPU2.9
- net PA10_CPU6: now also CPU.PB10; no longer CPU2.15
- net PA10_CPU7: now also CPU.PB0; no longer CPU2.13
- net PA10_GPU: now also GPU.PA10; no longer GPU1.7
- net PA11_GPU: now also GPU.PA11; no longer GPU1.8
- net PA12_GPU: now also GPU.PA12; no longer GPU1.9
- net PA15_GPU: now also GPU.PA15; no longer GPU1.10
- net PA1_GPU: now also GPU.PA1; no longer GPU.6
- net PA2_GPU: now also GPU.PA2; no longer GPU.7
- net PA3_GPU: now also GPU.PA3; no longer GPU.8
- net PA8_CPU: now also CPU.PA8; no longer CPU.5
- net PA9_CPU: now also CPU.PA9; no longer CPU.6
- net PA9_CPU1: now also CPU.PA11; no longer CPU.8
- net PA9_CPU2: now also CPU.PA3; no longer CPU2.8
- net PA9_CPU3: now also CPU.PA1; no longer CPU2.6
- net PA9_CPU4: now also CPU.PA7; no longer CPU2.12
- net PA9_CPU5: now also CPU.PA5; no longer CPU2.10
- net PA9_CPU6: now also CPU.PB11; no longer CPU2.16
- net PA9_CPU7: now also CPU.PB1; no longer CPU2.14
- net PA9_GPU: now also GPU.PA9; no longer GPU1.6
- net PB15_GPU: now also GPU.PB15; no longer GPU1.4
- net PB3_GPU: now also GPU.PB3; no longer GPU1.11
- net PB4_GPU: now also GPU.PB4; no longer GPU1.12
- net PB6_CPU: now also CPU.PB6; no longer CPU.14
- net PB7_CPU: now also CPU.PB7; no longer CPU.15
- net PB8_CPU: now also CPU.PB8; no longer CPU.16
- net PB8_GPU: now also GPU.PB8; no longer GPU1.16
- net PB9_CPU: now also CPU.PB9; no longer CPU.17
- net PB9_GPU: now also GPU.PB9; no longer GPU1.17
- net PC13_CPU: now also CPU.PC13; no longer CPU2.2
- net PC13_GPU: now also GPU.PC13; no longer GPU.2
- net PC14_GPU: now also GPU.PC14; no longer GPU.3
- net RED_LSP: now also GPU.PB11; no longer GPU.16
- net RED_MMSP: now also GPU.PB10; no longer GPU.15
- net RED_MSP: now also GPU.PB1; no longer GPU.14
- net RESET_CPU: now also CPU.RESET; no longer CPU2.17
- net RESET_GPU: now also GPU.RESET; no longer GPU.17
- net RIGHT: now also IC3A.D0, JP13.2, R65.1; no longer IC4A.D0
- net SELECT: now also IC3A.D4, JP1.2, R61.1; no longer IC4A.D4
- net START: now also IC3A.D5, JP2.2, R62.1; no longer IC4A.D5
- net UP: now also IC3A.D3; no longer IC4A.D3
- net VBAT_CPU: now also CPU.VBAT; no longer CPU2.1
- net VBAT_GPU: now also GPU.VBAT; no longer GPU.1
- net VSYNC: now also GPU.PB0; no longer GPU.13
Other:
- moved on the sheet: C1, C2, C23, C25, C28, C29, C3, C30, C31, C32, C33, C34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

Commit message: Board almost finished
Parts:
- removed C25, C28, C29, C30, C31, C32, C33, C34, C35, C36, C37: 100nF, deto:C1
- removed JP1, JP10, JP11, JP12, JP13, JP2, JP3, JP9: (no value), pinhead:PINHD-1X2
- removed JP4, JP5, JP6, JP7: (no value), pinhead:PINHD-1X3
- removed JP8: (no value), pinhead:PINHD-1X4
- removed R26, R27, R28, R29, R30, R31, R32, R33, R34, R35, R36, R37, R38, R39, R40, R41, R42, R43, R44, R45, R46, R47, R48, R49, R50, R51, R52, R53: 1k, rcl:R-EU_R0805
- added 3V3: +3V3, pinhead:PINHD-1X1
- added 5V: +5V, pinhead:PINHD-1X1
- added A, B, DOWN, LEFT, RIGHT, SELECT, START, UP: MOMENTARY-SWITCH-SPST-PTH-12MM, SparkFun-Switches:MOMENTARY-SWITCH-SPST-PTH-12MM
- added C12, C13, C14, C15, C16, C17, C18, C19, C20, C21, C22: 100nF, rcl:C-EUC0805
- added C_DATA_1, C_DATA_2, C_DATA_3, C_DATA_4: (no value), pinhead:PINHD-1X3
- added GND: GND, pinhead:PINHD-1X1
- added GNDA: GNDA, pinhead:PINHD-1X1
- added VCC: VCC, pinhead:PINHD-1X1
- C1, C2, C23, C3, C4, C5, C6, C7: device deto:C1 -> rcl:C-EUC0805
- renumbered JP14 to CLOCK, JP15 to COUNTER
Connections:
- net SDCARDCLK renamed SDCLK
- net SDCARDCMD renamed SDCMD
- net SDCARDHOTPLUG renamed SDHP
- net SDCARDIN renamed SDIN
- net SDCARDOUT renamed SDOUT
- removed net N$10: JP4.3, JP8.4
- removed net N$6 (its old number): JP7.3, JP8.1
- removed net N$7: JP6.3, JP8.2
- removed net N$9: JP5.3, JP8.3
- removed net PA0_GPU: C28.2, GPU.PA0, R45.1
- removed net PA10_CPU2: CPU.PA2, R27.1
- removed net PA10_CPU3: CPU.PA0, R29.1
- removed net PA10_CPU4: CPU.PA6, R31.1
- removed net PA10_CPU5: CPU.PA4, R33.1
- removed net PA10_CPU6: CPU.PB10, R35.1
- removed net PA10_CPU7: CPU.PB0, R37.1
- removed net PA10_GPU: C30.2, GPU.PA10, R47.2
- removed net PA11_GPU: C33.2, GPU.PA11, R48.2
- removed net PA12_GPU: C32.2, GPU.PA12, R49.2
- removed net PA1_GPU: C29.2, GPU.PA1, R44.1
- removed net PA2_GPU: C23.2, GPU.PA2, R43.1
- removed net PA3_GPU: C25.2, GPU.PA3, R42.1
- removed net PA9_CPU2: CPU.PA3, R26.1
- removed net PA9_CPU3: CPU.PA1, R28.1
- removed net PA9_CPU4: CPU.PA7, R30.1
- removed net PA9_CPU5: CPU.PA5, R32.1
- removed net PA9_CPU6: CPU.PB11, R34.1
- removed net PA9_CPU7: CPU.PB1, R36.1
- removed net PA9_GPU: C31.2, GPU.PA9, R46.2
- removed net PB3_GPU: C35.2, GPU.PB3, R50.2
- removed net PB4_GPU: C34.2, GPU.PB4, R51.2
- removed net PB6_CPU: CPU.PB6, R41.1
- removed net PB7_CPU: CPU.PB7, R40.1
- removed net PB8_CPU: CPU.PB8, R39.1
- removed net PB8_GPU: C37.2, GPU.PB8, R52.2
- removed net PB9_CPU: CPU.PB9, R38.1
- removed net PB9_GPU: C36.2, GPU.PB9, R53.2
- net +3V3: now also 3V3.1, C6.1; no longer C6.2
- net +5V: now also 5V.1, C1.1, C2.1, C3.1, C4.1, C5.1; no longer C1.2, C2.2, C3.2, C4.2, C5.2
- net A: now also A.2; no longer JP9.2
- net B: now also B.2; no longer JP3.2
- net C1: now also C_DATA_1.2; no longer JP4.2
- net C1_DATA: now also C_DATA_1.1; no longer JP4.1
- net C2: now also C_DATA_2.2; no longer JP5.2
- net C2_DATA: now also C_DATA_2.1; no longer JP5.1
- net C3: now also C_DATA_3.2; no longer JP6.2
- net C3_DATA: now also C_DATA_3.1; no longer JP6.1
- net C4: now also C_DATA_4.2; no longer JP7.2
- net C4_DATA: now also C_DATA_4.1; no longer JP7.1
- net DOUBLE1: now also C21.1, GPU.PB4; no longer R51.1
- net DOUBLE2: now also C23.1, GPU.PB9; no longer R53.1
- net DOWN: now also DOWN.2; no longer JP11.2
- net GND: now also C1.2, C12.2, C13.2, C14.2, C15.2, C16.2, C17.2, C18.2, C19.2, C2.2, C20.2, C21.2, C22.2, C23.2, C3.2, C4.2, C5.2, C6.2, GND.1; no longer C1.1, C2.1, C23.1, C25.1, C28.1, C29.1, C3.1, C30.1, C31.1, C32.1, C33.1, C34.1, C35.1, C36.1, C37.1, C4.1, C5.1, C6.1, C7.1, CONTROLLER-IN.GND, CONTROLLER-IN.GND1, CONTROLLER-IN.SBU1, CONTROLLER-IN.SHIELD, CONTROLLER-IN.SHIELD1, CONTROLLER-IN.SSRXN2, CONTROLLER-IN.SSRXP2, CONTROLLER-IN.SSTXN1, CONTROLLER-IN.SSTXP1, R70.1
- net GNDA: now also C7.2, CONTROLLER-IN.GND, CONTROLLER-IN.GND1, CONTROLLER-IN.SBU1, CONTROLLER-IN.SHIELD, CONTROLLER-IN.SHIELD1, CONTROLLER-IN.SSRXN2, CONTROLLER-IN.SSRXP2, CONTROLLER-IN.SSTXN1, CONTROLLER-IN.SSTXP1, GNDA.1, R70.1
- net HOT_PLUG1: now also C20.1, GPU.PB3; no longer R50.1
- net HOT_PLUG2: now also C22.1, GPU.PB8; no longer R52.1
- net ID0_1: now also C15.1, GPU.PA0; no longer R45.2
- net ID0_2: now also C19.1, GPU.PA12; no longer R49.1
- net ID1_1: now also C14.1, GPU.PA1; no longer R44.2
- net ID1_2: now also C18.1, GPU.PA11; no longer R48.1
- net ID2_1: now also C13.1, GPU.PA2; no longer R43.2
- net ID2_2: now also C17.1, GPU.PA10; no longer R47.1
- net ID3_1: now also C12.1, GPU.PA3; no longer R42.2
- net ID3_2: now also C16.1, GPU.PA9; no longer R46.1
- net LEFT: now also LEFT.2; no longer JP12.2
- net RIGHT: now also RIGHT.2; no longer JP13.2
- net SELECT: now also SELECT.2; no longer JP1.2
- net SIG0_1: now also CPU.PA0; no longer R29.2
- net SIG0_2: now also CPU.PB0; no longer R37.2
- net SIG1_1: now also CPU.PA1; no longer R28.2
- net SIG1_2: now also CPU.PB1; no longer R36.2
- net SIG2_1: now also CPU.PA2; no longer R27.2
- net SIG2_2: now also CPU.PB10; no longer R35.2
- net SIG3_1: now also CPU.PA3; no longer R26.2
- net SIG3_2: now also CPU.PB11; no longer R34.2
- net SIG4_1: now also CPU.PA4; no longer R33.2
- net SIG4_2: now also CPU.PB9; no longer R38.2
- net SIG5_1: now also CPU.PA5; no longer R32.2
- net SIG5_2: now also CPU.PB8; no longer R39.2
- net SIG6_1: now also CPU.PA6; no longer R31.2
- net SIG6_2: now also CPU.PB7; no longer R40.2
- net SIG7_1: now also CPU.PA7; no longer R30.2
- net SIG7_2: now also CPU.PB6; no longer R41.2
- net START: now also START.2; no longer JP2.2
- net UP: now also UP.2; no longer JP10.2
- net VCC: now also A.1, B.1, C7.1, DOWN.1, LEFT.1, RIGHT.1, SELECT.1, START.1, UP.1, VCC.1; no longer C7.2, JP1.1, JP10.1, JP11.1, JP12.1, JP13.1, JP2.1, JP3.1, JP9.1
Other:
- moved on the sheet: C10, C11, C8, C9, IC1D, IC1P, IC2P, IC3P, IC4P, POWER-IN, R1, R2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

Commit message: set board labels and fixed errors
Connections:
- net GND: no longer POWER-IN.SHIELD, POWER-IN.SHIELD1, USB-CONTROLLER1.SHIELD, USB-CONTROLLER1.SHIELD1, USB-CONTROLLER2.SHIELD, USB-CONTROLLER2.SHIELD1, USB-CONTROLLER3.SHIELD, USB-CONTROLLER3.SHIELD1, USB-CONTROLLER4.SHIELD, USB-CONTROLLER4.SHIELD1
- net GNDA: no longer CONTROLLER-IN.SHIELD, CONTROLLER-IN.SHIELD1
Changed lines of the file:
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@@
 <net name="GND" class="0">
 <segment>
-<wire x1="26.67" y1="140.97" x2="26.67" y2="143.51" width="0.1524" layer="91"/>
 <wire x1="29.21" y1="146.05" x2="26.67" y2="146.05" width="0.1524" layer="91"/>
 <wire x1="26.67" y1="146.05" x2="26.67" y2="148.59" width="0.1524" layer="91"/>
@@
 <wire x1="26.67" y1="148.59" x2="29.21" y2="148.59" width="0.1524" layer="91"/>
 <junction x="26.67" y="148.59"/>
-<wire x1="26.67" y1="146.05" x2="26.67" y2="143.51" width="0.1524" layer="91"/>
+<wire x1="26.67" y1="146.05" x2="26.67" y2="140.97" width="0.1524" layer="91"/>
 <junction x="26.67" y="146.05"/>
-<wire x1="26.67" y1="143.51" x2="29.21" y2="143.51" width="0.1524" layer="91"/>
-<junction x="26.67" y="143.51"/>
 <pinref part="USB-CONTROLLER3" gate="G$1" pin="SBU1"/>
 <pinref part="USB-CONTROLLER3" gate="G$1" pin="SSRXN2"/>
 <pinref part="USB-CONTROLLER3" gate="G$1" pin="SSRXP2"/>
-<pinref part="USB-CONTROLLER3" gate="G$1" pin="SHIELD"/>
 <wire x1="26.67" y1="151.13" x2="26.67" y2="161.29" width="0.1524" layer="91"/>
 <junction x="26.67" y="151.13"/>
@@
 </segment>
 <segment>
-<wire x1="67.31" y1="143.51" x2="67.31" y2="146.05" width="0.1524" layer="91"/>
 <wire x1="67.31" y1="146.05" x2="67.31" y2="148.59" width="0.1524" layer="91"/>
 <wire x1="67.31" y1="148.59" x2="64.77" y2="148.59" width="0.1524" layer="91"/>
 <wire x1="64.77" y1="146.05" x2="67.31" y2="146.05" width="0.1524" layer="91"/>
 <junction x="67.31" y="146.05"/>
-<wire x1="64.77" y1="143.51" x2="67.31" y2="143.51" width="0.1524" layer="91"/>
-<junction x="67.31" y="143.51"/>
-<wire x1="67.31" y1="140.97" x2="67.31" y2="143.51" width="0.1524" layer="91"/>
+<wire x1="67.31" y1="140.97" x2="67.31" y2="146.05" width="0.1524" layer="91"/>
 <pinref part="USB-CONTROLLER3" gate="G$1" pin="GND"/>
 <pinref part="USB-CONTROLLER3" gate="G$1" pin="GND1"/>
-<pinref part="USB-CONTROLLER3" gate="G$1" pin="SHIELD1"/>
 <pinref part="GND9" gate="1" pin="GND"/>
 </segment>
@@
 <pinref part="USB-CONTROLLER2" gate="G$1" pin="SBU1"/>
 <wire x1="115.57" y1="151.13" x2="113.03" y2="151.13" width="0.1524" layer="91"/>
-<pinref part="USB-CONTROLLER2" gate="G$1" pin="SHIELD"/>
-<wire x1="115.57" y1="143.51" x2="113.03" y2="143.51" width="0.1524" layer="91"/>
-<wire x1="113.03" y1="143.51" x2="113.03" y2="146.05" width="0.1524" layer="91"/>
 <junction x="113.03" y="146.05"/>
-<wire x1="113.03" y1="140.97" x2="113.03" y2="143.51" width="0.1524" layer="91"/>
-<junction x="113.03" y="143.51"/>
+<wire x1="113.03" y1="140.97" x2="113.03" y2="146.05" width="0.1524" layer="91"/>
 <wire x1="113.03" y1="151.13" x2="113.03" y2="161.29" width="0.1524" layer="91"/>
 <junction x="113.03" y="151.13"/>
@@
 </segment>
 <segment>
-<wire x1="153.67" y1="143.51" x2="153.67" y2="146.05" width="0.1524" layer="91"/>
 <wire x1="153.67" y1="146.05" x2="153.67" y2="148.59" width="0.1524" layer="91"/>
 <wire x1="153.67" y1="148.59" x2="151.13" y2="148.59" width="0.1524" layer="91"/>
 <wire x1="151.13" y1="146.05" x2="153.67" y2="146.05" width="0.1524" layer="91"/>
 <junction x="153.67" y="146.05"/>
-<wire x1="151.13" y1="143.51" x2="153.67" y2="143.51" width="0.1524" layer="91"/>
-<junction x="153.67" y="143.51"/>
-<wire x1="153.67" y1="140.97" x2="153.67" y2="143.51" width="0.1524" layer="91"/>
+<wire x1="153.67" y1="140.97" x2="153.67" y2="146.05" width="0.1524" layer="91"/>
 <pinref part="USB-CONTROLLER2" gate="G$1" pin="GND"/>
 <pinref part="USB-CONTROLLER2" gate="G$1" pin="GND1"/>
-<pinref part="USB-CONTROLLER2" gate="G$1" pin="SHIELD1"/>
 <pinref part="GND16" gate="1" pin="GND"/>
 </segment>
 <segment>
-<wire x1="153.67" y1="101.6" x2="153.67" y2="104.14" width="0.1524" layer="91"/>
 <wire x1="153.67" y1="104.14" x2="153.67" y2="106.68" width="0.1524" layer="91"/>
 <wire x1="153.67" y1="106.68" x2="151.13" y2="106.68" width="0.1524" layer="91"/>
 <wire x1="151.13" y1="104.14" x2="153.67" y2="104.14" width="0.1524" layer="91"/>
 <junction x="153.67" y="104.14"/>
-<wire x1="151.13" y1="101.6" x2="153.67" y2="101.6" width="0.1524" layer="91"/>
-<junction x="153.67" y="101.6"/>
-<wire x1="153.67" y1="99.06" x2="153.67" y2="101.6" width="0.1524" layer="91"/>
+<wire x1="153.67" y1="99.06" x2="153.67" y2="104.14" width="0.1524" layer="91"/>
 <pinref part="USB-CONTROLLER1" gate="G$1" pin="GND"/>
 <pinref part="USB-CONTROLLER1" gate="G$1" pin="GND1"/>
-<pinref part="USB-CONTROLLER1" gate="G$1" pin="SHIELD1"/>
 <pinref part="GND17" gate="1" pin="GND"/>
 </segment>
@@
 <wire x1="113.03" y1="104.14" x2="113.03" y2="106.68" width="0.1524" layer="91"/>
 <junction x="113.03" y="104.14"/>
-<wire x1="113.03" y1="99.06" x2="113.03" y2="101.6" width="0.1524" layer="91"/>
-<pinref part="USB-CONTROLLER1" gate="G$1" pin="SHIELD"/>
-<wire x1="113.03" y1="101.6" x2="113.03" y2="104.14" width="0.1524" layer="91"/>
-<wire x1="115.57" y1="101.6" x2="113.03" y2="101.6" width="0.1524" layer="91"/>
-<junction x="113.03" y="101.6"/>
+<wire x1="113.03" y1="99.06" x2="113.03" y2="104.14" width="0.1524" layer="91"/>
 <wire x1="113.03" y1="109.22" x2="113.03" y2="119.38" width="0.1524" layer="91"/>
 <junction x="113.03" y="109.22"/>
@@
 </segment>
 <segment>
-<wire x1="69.85" y1="101.6" x2="69.85" y2="104.14" width="0.1524" layer="91"/>
 <wire x1="69.85" y1="104.14" x2="69.85" y2="106.68" width="0.1524" layer="91"/>
 <wire x1="69.85" y1="106.68" x2="67.31" y2="106.68" width="0.1524" layer="91"/>
 <wire x1="67.31" y1="104.14" x2="69.85" y2="104.14" width="0.1524" layer="91"/>
 <junction x="69.85" y="104.14"/>
-<wire x1="67.31" y1="101.6" x2="69.85" y2="101.6" width="0.1524" layer="91"/>
-<junction x="69.85" y="101.6"/>
-<wire x1="69.85" y1="99.06" x2="69.85" y2="101.6" width="0.1524" layer="91"/>
+<wire x1="69.85" y1="99.06" x2="69.85" y2="104.14" width="0.1524" layer="91"/>
 <pinref part="USB-CONTROLLER4" gate="G$1" pin="GND"/>
 <pinref part="USB-CONTROLLER4" gate="G$1" pin="GND1"/>
-<pinref part="USB-CONTROLLER4" gate="G$1" pin="SHIELD1"/>
 <pinref part="GND21" gate="1" pin="GND"/>
 </segment>
@@
 <wire x1="29.21" y1="104.14" x2="29.21" y2="106.68" width="0.1524" layer="91"/>
 <junction x="29.21" y="104.14"/>
-<wire x1="29.21" y1="99.06" x2="29.21" y2="101.6" width="0.1524" layer="91"/>
-<wire x1="29.21" y1="101.6" x2="29.21" y2="104.14" width="0.1524" layer="91"/>
+<wire x1="29.21" y1="99.06" x2="29.21" y2="104.14" width="0.1524" layer="91"/>
 <wire x1="29.21" y1="109.22" x2="29.21" y2="119.38" width="0.1524" layer="91"/>
 <junction x="29.21" y="109.22"/>
@@
 <wire x1="31.75" y1="119.38" x2="29.21" y2="119.38" width="0.1524" layer="91"/>
 <junction x="29.21" y="119.38"/>
-<pinref part="USB-CONTROLLER4" gate="G$1" pin="SHIELD"/>
-<wire x1="31.75" y1="101.6" x2="29.21" y2="101.6" width="0.1524" layer="91"/>
-<junction x="29.21" y="101.6"/>
 <pinref part="GND22" gate="1" pin="GND"/>
 </segment>
@@
 <wire x1="353.06" y1="134.62" x2="353.06" y2="137.16" width="0.1524" layer="91"/>
 <junction x="353.06" y="134.62"/>
-<pinref part="POWER-IN" gate="G$1" pin="SHIELD1"/>
-<wire x1="353.06" y1="132.08" x2="350.52" y2="132.08" width="0.1524" layer="91"/>
-<wire x1="353.06" y1="132.08" x2="353.06" y2="134.62" width="0.1524" layer="91"/>
-<wire x1="353.06" y1="129.54" x2="353.06" y2="132.08" width="0.1524" layer="91"/>
-<junction x="353.06" y="132.08"/>
+<wire x1="353.06" y1="129.54" x2="353.06" y2="134.62" width="0.1524" layer="91"/>
 <pinref part="GND37" gate="1" pin="GND"/>
 </segment>
@@
 <pinref part="POWER-IN" gate="G$1" pin="SSRXN2"/>
 <wire x1="312.42" y1="129.54" x2="312.42" y2="132.08" width="0.1524" layer="91"/>
-<wire x1="314.96" y1="132.08" x2="312.42" y2="132.08" width="0.1524" layer="91"/>
-<pinref part="POWER-IN" gate="G$1" pin="SHIELD"/>
 <wire x1="312.42" y1="137.16" x2="312.42" y2="134.62" width="0.1524" layer="91"/>
 <junction x="312.42" y="132.08"/>
@@
 <wire x1="77.47" y1="127" x2="77.47" y2="129.54" width="0.1524" layer="91"/>
 <junction x="77.47" y="127"/>
-<pinref part="CONTROLLER-IN" gate="G$1" pin="SHIELD1"/>
-<wire x1="77.47" y1="124.46" x2="74.93" y2="124.46" width="0.1524" layer="91"/>
-<wire x1="77.47" y1="124.46" x2="77.47" y2="127" width="0.1524" layer="91"/>
-<wire x1="77.47" y1="121.92" x2="77.47" y2="124.46" width="0.1524" layer="91"/>
-<junction x="77.47" y="124.46"/>
+<wire x1="77.47" y1="121.92" x2="77.47" y2="127" width="0.1524" layer="91"/>
 <pinref part="GND2" gate="1" pin="GNDA"/>
 </segment>
@@
 <pinref part="CONTROLLER-IN" gate="G$1" pin="SSRXN2"/>
 <wire x1="36.83" y1="121.92" x2="36.83" y2="124.46" width="0.1524" layer="91"/>
-<wire x1="39.37" y1="124.46" x2="36.83" y2="124.46" width="0.1524" layer="91"/>
-<pinref part="CONTROLLER-IN" gate="G$1" pin="SHIELD"/>
 <wire x1="36.83" y1="129.54" x2="36.83" y2="127" width="0.1524" layer="91"/>
 <junction x="36.83" y="124.46"/>
