File: eagle/mainboard.sch (EAGLE design)
At the start: 100 parts, among them IC1 74HC02D, IC2 74HC151D, IC3 74HC151D, IC4 74HC590D

Commit message: usb change
Parts:
- removed CONTROLLER-IN, POWER-IN, USB-CONTROLLER1, USB-CONTROLLER2, USB-CONTROLLER3, USB-CONTROLLER4: 632723100011_USBC_3.1, Eagle_WR-USB (rev22c):632723100011_USBC_3.1
- removed R55, R70: 5k1Ω, rcl:R-EU_R0805
- removed R57, R58, R59, R60: 56kΩ, rcl:R-EU_R0805
- added USBC1-2, USB_C3-4: 61400826021, Wurth_Connectors_WR-USB:61400826021
- added USBCIN, USBPOWER: 61410416121R, Wurth_Connectors_WR-USB:61410416121R
Connections:
- removed net N$1: POWER-IN.VBUS, POWER-IN.VBUS1, R5.1
- removed net N$13: R58.2, USB-CONTROLLER4.CC
- removed net N$14: R59.2, USB-CONTROLLER3.CC
- removed net N$31: R60.2, USB-CONTROLLER2.CC
- removed net N$32: CONTROLLER-IN.VBUS, CONTROLLER-IN.VBUS1, R71.1
- removed net N$33: CONTROLLER-IN.CC, R70.2
- removed net N$6: R57.2, USB-CONTROLLER1.CC
- new net N$7: R1.1, USB_C3-4USBA.VBUS
- net +5V: no longer R57.1, R58.1, R59.1, R60.1
- net C1_DATA: now also USBC1-2USBA.D-; no longer USB-CONTROLLER1.DP1
- net C2_DATA: now also USBC1-2USBB.D-; no longer USB-CONTROLLER2.DP1
- net C3_DATA: now also USB_C3-4USBA.D-; no longer USB-CONTROLLER3.DP1
- net C4_DATA: now also USB_C3-4USBB.D-; no longer USB-CONTROLLER4.DP1
- net CONTROLLER_CLOCK: now also USBCIN.D+; no longer CONTROLLER-IN.DN1
- net CONTROLLER_OUT: now also USBCIN.D-; no longer CONTROLLER-IN.DP1
- net C_CLOCK: now also USBC1-2USBA.D+, USBC1-2USBB.D+, USB_C3-4USBA.D+, USB_C3-4USBB.D+; no longer USB-CONTROLLER1.DN1, USB-CONTROLLER2.DN1, USB-CONTROLLER3.DN1, USB-CONTROLLER4.DN1
- net GND: now also USBC1-2USBA.GND, USBC1-2USBA.SHIELD, USBC1-2USBB.GND, USBC1-2USBB.SHIELD, USBPOWER.GND, USBPOWER.SHIELD, USB_C3-4USBA.GND, USB_C3-4USBA.SHIELD, USB_C3-4USBB.GND, USB_C3-4USBB.SHIELD; no longer POWER-IN.DN1, POWER-IN.DP1, POWER-IN.GND, POWER-IN.GND1, POWER-IN.SBU1, POWER-IN.SSRXN2, POWER-IN.SSRXP2, POWER-IN.SSTXN1, POWER-IN.SSTXP1, R55.1, USB-CONTROLLER1.GND, USB-CONTROLLER1.GND1, USB-CONTROLLER1.SBU1, USB-CONTROLLER1.SSRXN2, USB-CONTROLLER1.SSRXP2, USB-CONTROLLER1.SSTXN1, USB-CONTROLLER1.SSTXP1, USB-CONTROLLER2.GND, USB-CONTROLLER2.GND1, USB-CONTROLLER2.SBU1, USB-CONTROLLER2.SSRXN2, USB-CONTROLLER2.SSRXP2, USB-CONTROLLER2.SSTXN1, USB-CONTROLLER2.SSTXP1, USB-CONTROLLER3.GND, USB-CONTROLLER3.GND1, USB-CONTROLLER3.SBU1, USB-CONTROLLER3.SSRXN2, USB-CONTROLLER3.SSRXP2, USB-CONTROLLER3.SSTXN1, USB-CONTROLLER3.SSTXP1, USB-CONTROLLER4.GND, USB-CONTROLLER4.GND1, USB-CONTROLLER4.SBU1, USB-CONTROLLER4.SSRXN2, USB-CONTROLLER4.SSRXP2, USB-CONTROLLER4.SSTXN1, USB-CONTROLLER4.SSTXP1
- net GNDA: now also USBCIN.GND, USBCIN.SHIELD; no longer CONTROLLER-IN.GND, CONTROLLER-IN.GND1, CONTROLLER-IN.SBU1, CONTROLLER-IN.SSRXN2, CONTROLLER-IN.SSRXP2, CONTROLLER-IN.SSTXN1, CONTROLLER-IN.SSTXP1, R70.1
- net N$2: now also USBC1-2USBB.VBUS; no longer USB-CONTROLLER2.VBUS, USB-CONTROLLER2.VBUS1
- net N$3: now also R4.1, USB_C3-4USBB.VBUS; no longer R1.1, USB-CONTROLLER3.VBUS, USB-CONTROLLER3.VBUS1
- net N$4: now also R3.1, USBC1-2USBA.VBUS; no longer R4.1, USB-CONTROLLER4.VBUS, USB-CONTROLLER4.VBUS1
- net N$5: now also R71.1, USBCIN.VBUS; no longer R3.1, USB-CONTROLLER1.VBUS, USB-CONTROLLER1.VBUS1
- net N$8: now also R5.1, USBPOWER.VBUS; no longer POWER-IN.CC, R55.2
Other:
- moved on the sheet: C1, C2, C3, C4, C5, C7, R1, R2, R3, R4, R5, R71

Commit message: Work in progress board rework
Parts:
- removed C12, C13, C14, C15, C16, C17, C18, C19, C20, C21, C22, C23: 100nF, rcl:C-EUC0805
- removed C_DATA_1, C_DATA_2, C_DATA_3, C_DATA_4: (no value), pinhead:PINHD-1X3
- added CLOCK1: (no value), pinhead:PINHD-1X1
Connections:
- net C1: no longer C_DATA_1.2
- net C1_DATA: no longer C_DATA_1.1
- net C2: no longer C_DATA_2.2
- net C2_DATA: no longer C_DATA_2.1
- net C3: no longer C_DATA_3.2
- net C3_DATA: no longer C_DATA_3.1
- net C4: no longer C_DATA_4.2
- net C4_DATA: no longer C_DATA_4.1
- net CONTROLLER_OUT: now also CLOCK1.1
- net DOUBLE1: no longer C21.1
- net DOUBLE2: no longer C23.1
- net GND: no longer C12.2, C13.2, C14.2, C15.2, C16.2, C17.2, C18.2, C19.2, C20.2, C21.2, C22.2, C23.2
- net HOT_PLUG1: no longer C20.1
- net HOT_PLUG2: no longer C22.1
- net ID0_1: no longer C15.1
- net ID0_2: no longer C19.1
- net ID1_1: no longer C14.1
- net ID1_2: no longer C18.1
- net ID2_1: no longer C13.1
- net ID2_2: no longer C17.1
- net ID3_1: no longer C12.1
- net ID3_2: no longer C16.1
